File: CAD/BSS_T10 Underboard component design.sch (EAGLE design)
At the start: 10 parts

Commit message: board
Parts:
- removed SWITCH: BSS123, transistor-small-signal:BSS123
- removed VREG: 7805T, linear:7805T
- added IC1: 7805DT, linear:7805DT
- C3: value .1pF -> .1uF
- R1: value (none) -> 1k
- TO_SEN, VOLT_IN: value (none) -> MA03-1
- renumbered CBP1 to C3, LED1 to LED
Connections:
- net N$3 renamed RLED
- removed net BATTERY: SWITCH.D, VOLT_IN.3
- removed net N$2: C2.1
- removed net N$8: AVR.PB2/PCINT2/SCK/ADC1/T0, TO_SEN.2
- new net 12VBATTERY: C2.1, IC1.VI, VOLT_IN.2
- net +5V: now also IC1.VO; no longer VREG.VO
- net GND: now also IC1.GND, TO_SEN.2; no longer TO_SEN.1, VREG.GND
- net N$1: now also AVR.PB4/PCINT4/ADC2, TO_SEN.1; no longer SWITCH.S, VREG.VI
- net N$4: now also AVR.PB0/PCINT0/AIN0/OC0A/MOSI; no longer AVR.PB4/PCINT4/ADC2
- net TSIG: now also AVR.PB2/PCINT2/SCK/ADC1/T0, VOLT_IN.3; no longer SWITCH.G, VOLT_IN.2
Other:
- note added: "ATTINY Programmed off board in Aurduino"
- note added: "Connects to car battery (12V), turn signal (logic signal) and GND"
- note added: "Connects to ultrasonic sensors power, ground and analog output pins"
- note added: "Test pin"
- note removed: "12v battery"
- note removed: "AnOut_Sensor"
- note removed: "turn sig"
- moved on the sheet: TO_SEN, VOLT_IN
